File: KiCad/Buttons/Buttons.kicad_pcb (KiCad board)
At the start: 2 copper layers, 38.4 x 23.6 mm, 15 parts, among them J1 KEYB, SW1 SET, SW2 OK, SW3 UP, SW4 RHT, SW5 DWN, SW6 LFT

Commit message: ver 2156
Many Updates
Parts:
- added D1: LED, LED_THT:LED_D3.0mm, F.Cu at (142.0, 79.2)
- added R7: R, Resistor_SMD:R_0805_2012Metric, F.Cu at (135.9, 76.7)
- R1: value R -> 910
- R2: value R -> 330
- R3: value R -> 680
- R4: value R -> 0
- R5: value R -> 1200
- R6: value R -> 1500
Connections:
- net Net-(J1-Pad3) renamed /AKB
- J1 pad 2: Net-(J1-Pad2) -> /5V
Routing:
- net Net-(D1-Pad1): track 0.00 -> 6.62 mm
- net GNDREF: track 88.2 -> 93.1 mm
- net /5V: track 0.00 -> 2.86 mm
- net Net-(J1-Pad2): track 2.54 -> 0.00 mm
