File: SD23CF/kicad/Tode-Backplane-SD23CF/AMPE32T30.kicad_pcb (KiCad board)
At the start: 2 copper layers, 39.1 x 75.2 mm, 26 parts, among them J1 PWR, J10 IN, J11 IO, J12 Batt, J13 13, J14 14, J15 15, J16 16, J17 Batt, J2 ICSP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

Commit message: SD23CF and BD241S
Obsolete SA212K
Other:
- net class Default removed
- net class Power removed
